File: ecad/displayport-switch.kicad_pcb (KiCad board)
At the start: 4 copper layers, 47 parts, among them P1 MOLEX_47272-0001, P2 MOLEX_47272-0001, P3 MOLEX_47272-0001, P4 CONN_01X03, P5 CONN_01X06, U1 HD3SS215IRTQT, U2 AP2112K-3.3

Commit message: Partial routing concepts
Parts:
- removed TEST1, TEST2, TEST3: CLIP_HOOK_WHITE, Applidyne_Test:KEYSTONE_5002
- P3: moved to B.Cu
- moved U2 94.7 mm to (142.3, 145.1)
- moved P5 93.8 mm to (153.5, 144.2)
- moved R15 88.9 mm to (168.8, 143.2)
- moved R13 88.8 mm to (162.6, 145.8)
- moved R14 87.2 mm to (168.8, 141.8)
- moved P4 84.2 mm to (152.0, 136.8), turned to 90 degrees
- moved P1 82.6 mm to (112.3, 119.5), turned to 180 degrees
- moved C18 76.2 mm to (137.4, 144.9)
- moved C19 74.9 mm to (137.2, 142.1)
- moved C3 69.2 mm to (120.6, 107.8)
- moved R8 67.9 mm to (168.3, 147.2)
- moved C7 65.0 mm to (120.6, 115.3), turned to 180 degrees
- moved C5 60.2 mm to (120.6, 116.5), turned to 180 degrees
- moved R1 59.0 mm to (120.6, 106.6), turned to 180 degrees
- moved P2 56.2 mm to (112.3, 95.5), turned to 180 degrees
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Connections:
- net Net-(C10-Pad1) renamed /_DC1+
- net Net-(C10-Pad2) renamed /DC1+
- net Net-(C11-Pad1) renamed /_DC2+
- net Net-(C11-Pad2) renamed /DC2+
- net Net-(C12-Pad1) renamed /_DC3+
- net Net-(C12-Pad2) renamed /DC3+
- net Net-(C13-Pad1) renamed /_DC0-
- net Net-(C13-Pad2) renamed /DC0-
- net Net-(C14-Pad1) renamed /_DC1-
- net Net-(C14-Pad2) renamed /DC1-
- net Net-(C15-Pad1) renamed /_DC2-
- net Net-(C15-Pad2) renamed /DC2-
- net Net-(C16-Pad1) renamed /_DC3-
- net Net-(C16-Pad2) renamed /DC3-
- net Net-(C5-Pad1) renamed /AUXA+
- net Net-(C5-Pad2) renamed /_AUXA+
- net Net-(C6-Pad1) renamed /AUXB+
- net Net-(C6-Pad2) renamed /_AUXB+
- net Net-(C7-Pad1) renamed /AUXA-
- net Net-(C7-Pad2) renamed /_AUXA-
- net Net-(C8-Pad1) renamed /AUXB-
- net Net-(C8-Pad2) renamed /_AUXB-
- net Net-(C9-Pad1) renamed /_DC0+
- net Net-(C9-Pad2) renamed /DC0+
- net Net-(P1-Pad1) renamed /DA0+
- net Net-(P1-Pad10) renamed /DA3+
- net Net-(P1-Pad12) renamed /DA3-
- net Net-(P1-Pad3) renamed /DA0-
- net Net-(P1-Pad4) renamed /DA1+
- net Net-(P1-Pad6) renamed /DA1-
- net Net-(P1-Pad7) renamed /DA2+
- net Net-(P1-Pad9) renamed /DA2-
- net Net-(P2-Pad1) renamed /DB0+
- net Net-(P2-Pad10) renamed /DB3+
- net Net-(P2-Pad12) renamed /DB3-
- net Net-(P2-Pad3) renamed /DB0-
- net Net-(P2-Pad4) renamed /DB1+
- net Net-(P2-Pad6) renamed /DB1-
- net Net-(P2-Pad7) renamed /DB2+
- net Net-(P2-Pad9) renamed /DB2-
- net Net-(P3-Pad15) renamed /AUXC+
- net Net-(P3-Pad17) renamed /AUXC-
Routing:
- net GND: track 0.00 -> 74.8 mm, vias 0 -> 24
- net /DA0+: track 0.00 -> 35.9 mm
- net /DA0-: track 0.00 -> 35.3 mm
- net /DA1+: track 0.00 -> 33.4 mm
- net /DA1-: track 0.00 -> 32.7 mm
- net /DA2+: track 0.00 -> 30.9 mm
- net /DA2-: track 0.00 -> 30.2 mm
- net /DA3+: track 0.00 -> 28.4 mm
- net /DA3-: track 0.00 -> 27.7 mm
- net /AUXC-: track 0.00 -> 15.3 mm, vias 0 -> 1
- net /AUXC+: track 0.00 -> 15.3 mm, vias 0 -> 1
- net /DB3+: track 0.00 -> 13.4 mm
- net /DB1+: track 0.00 -> 13.4 mm
- net /DB2+: track 0.00 -> 13.4 mm
- net /DB0+: track 0.00 -> 13.4 mm
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Other:
- board outline added: 60 x 45 mm
- net class Default: via_dia 0.8 -> 0.45; via_drill 0.4 -> 0.25

Commit message: HS routing done?
Parts:
- moved R13 36.5 mm to (139.9, 117.2)
- moved R14 36.5 mm to (146.2, 113.0)
- moved R15 36.5 mm to (146.2, 114.5)
- moved R8 36.5 mm to (145.8, 118.5)
- moved P4 21.4 mm to (164.9, 119.7), turned to 180 degrees
- moved U2 19.9 mm to (146.1, 125.5)
- moved C19 19.9 mm to (140.9, 122.5)
- moved C18 19.9 mm to (141.1, 125.3)
- moved P5 19.8 mm to (155.2, 124.5), turned to 180 degrees
- moved R4 14.7 mm to (140.3, 94.1)
- moved R6 12.5 mm to (140.3, 90.2), turned to 180 degrees
- moved R5 12.5 mm to (140.3, 88.9)
- moved R3 11.2 mm to (140.3, 92.4), turned to 180 degrees
- moved F2 6.46 mm to (127.0, 89.6)
- moved R12 6.00 mm to (120.7, 89.0)
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Routing:
- net Net-(C3-Pad1): track 0.00 -> 42.5 mm
- net Net-(C17-Pad1): track 0.00 -> 41.4 mm
- net Net-(C4-Pad1): track 0.00 -> 41.3 mm
- net Net-(P1-Pad18): track 1.52 -> 36.1 mm, vias 1 -> 2
- net /AUXA-: track 5.06 -> 32.0 mm, vias 0 -> 2
- net /AUXA+: track 5.74 -> 32.0 mm, vias 0 -> 2
- net Net-(P2-Pad18): track 2.03 -> 25.5 mm, vias 1 -> 0
- net Net-(P3-Pad13): track 0.00 -> 18.5 mm, vias 0 -> 1
- net Net-(P3-Pad14): track 0.00 -> 16.7 mm, vias 0 -> 1
- net Net-(F2-Pad1): track 0.00 -> 13.1 mm
- net ENABLE: track 1.93 -> 14.9 mm
- net /DA3-: track 27.7 -> 40.0 mm
- net Net-(F3-Pad1): track 0.00 -> 11.7 mm, vias 0 -> 1
- net /DA3+: track 28.4 -> 40.0 mm
- net Net-(P2-Pad13): track 6.65 -> 17.8 mm
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- added copper zone on In2.Cu, net +3.3V
- added copper zone on In1.Cu, net GND
Other:
- outline, holes or cut-outs redrawn

Commit message: Routing/Layout completed, cosmetics
Parts:
- removed P4: CONN_01X03, Applidyne_Connector_Wurth:61300311121
- C18, C19: value 10u_X7R_3216M -> 4u7_X5R_1608M; footprint Applidyne_Capacitor:CAPC3216X135N -> Applidyne_Capacitor:CAPC1608X90N
- moved R13 13.6 mm to (152.7, 112.3), turned to 180 degrees
- moved C19 13.2 mm to (152.7, 116.6)
- moved C18 11.6 mm to (152.7, 124.2)
- moved R8 10.2 mm to (152.7, 111.0)
- moved U2 8.32 mm to (152.7, 120.4)
- moved R14 6.74 mm to (152.7, 114.8)
- moved R15 6.58 mm to (152.7, 113.5), turned to 180 degrees
- moved P5 1.55 mm to (156.7, 124.2)
Connections:
- P5 pad 4: ENABLE -> INPUT_SELECT
- P5 pad 6: INPUT_SELECT -> ENABLE
Routing:
- net INPUT_SELECT: track 6.81 -> 35.2 mm
- net AUX_SEL: track 6.69 -> 33.0 mm
- net ENABLE: track 14.9 -> 40.6 mm
- net +5V: track 0.00 -> 21.0 mm
- net GND: track 83.6 -> 94.2 mm, vias 46 -> 50
- net +3.3V: track 19.6 -> 26.2 mm, vias 10 -> 15
Other:
- board text added: "3V3"
- board text added: "DP1.2 SWITCH S.RAPSON 2021"
- board text added: "ENABLE"
- board text added: "GND"
- board text added: "OUTPUT C"
- board text added: "SELECT"
- board text added: "SOURCE A"
- board text added: "SOURCE B"
- board text added: "VCC"
